Commit message: fix(assets): correct fixed-wing VTOL and UUV assets

File: acesim/env/mujoco/asset/advanced_plane/advanced_plane.urdf (robot description, URDF)
Before this commit: robot plane, 8 links, 7 joints
Links:
- link base_link: mass 1 -> 1.5; geometry collision box size=0.752 0.752 0.176; visual mesh filename=package://advanced_plane/meshes/base_link_visual_0.stl scale=0.0016 0.0016 0.0016
- link elevator: geometry visual mesh filename=package://advanced_plane/meshes/elevator_visual_0.stl scale=0.0016 0.0016 0.0016
- link left_elevon: geometry visual mesh filename=package://advanced_plane/meshes/left_elevon_visual_0.stl scale=0.0016 0.0016 0.0016
- link left_flap: geometry visual mesh filename=package://advanced_plane/meshes/left_flap_visual_0.stl scale=0.0016 0.0016 0.0016
- link right_elevon: geometry visual mesh filename=package://advanced_plane/meshes/right_elevon_visual_0.stl scale=0.0016 0.0016 0.0016
- link right_flap: geometry visual mesh filename=package://advanced_plane/meshes/right_flap_visual_0.stl scale=0.0016 0.0016 0.0016
- link rotor_4: geometry collision cylinder length=0.005 radius=0.0670132746; visual mesh filename=package://advanced_plane/meshes/rotor_4_vis.stl scale=0.52 0.52 0.52
- link rudder: geometry visual mesh filename=package://advanced_plane/meshes/rudder_visual_0.stl scale=0.0016 0.0016 0.0016
Joints:
- joint elevator_joint: limit lower=-0.78 upper=0.78 effort=1000 velocity=1000 -> lower=-0.53 upper=0.53 effort=1000 velocity=1000; origin xyz=-0.5 0 0 rpy=0 0 0 -> xyz=-0.8 0 0 rpy=0 0 0
- joint left_elevon_joint: limit lower=-0.78 upper=0.78 effort=1000 velocity=1000 -> lower=-0.53 upper=0.53 effort=1000 velocity=1000; origin xyz=-0.07 0.4 0.08 rpy=0 0 0 -> xyz=-0.112 0.64 0.128 rpy=0.00 0 0.0
- joint left_flap_joint: limit lower=-0.78 upper=0.78 effort=1000 velocity=1000 -> lower=-0.53 upper=0.53 effort=1000 velocity=1000; origin xyz=-0.07 0.2 0.08 rpy=0 0 0 -> xyz=-0.112 0.32 0.128 rpy=0.00 0 0.0
- joint right_elevon_joint: limit lower=-0.78 upper=0.78 effort=1000 velocity=1000 -> lower=-0.53 upper=0.53 effort=1000 velocity=1000; origin xyz=-0.07 -0.4 0.08 rpy=0 0 0 -> xyz=-0.112 -0.64 0.128 rpy=0.00 0 0.0
- joint right_flap_joint: limit lower=-0.78 upper=0.78 effort=1000 velocity=1000 -> lower=-0.53 upper=0.53 effort=1000 velocity=1000; origin xyz=-0.07 -0.2 0.08 rpy=0 0 0 -> xyz=-0.112 -0.32 0.128 rpy=0.00 0 0.0
- joint rotor_4_joint: origin xyz=0.3 0 0 rpy=0 0 0 -> xyz=0.202208044 0 -0.0802970325 rpy=0 1.57 0
- joint rudder_joint: limit lower=-0.78 upper=0.78 effort=1000 velocity=1000 -> lower=-0.53 upper=0.53 effort=1000 velocity=1000; origin xyz=-0.5 0 0.05 rpy=0 0 0 -> xyz=-0.8 0 0.08 rpy=0.00 0 0.0

File: acesim/env/mujoco/asset/standard_vtol/standard_vtol.urdf (robot description, URDF)
Before this commit: robot standard_vtol, 9 links, 8 joints
Links:
- added link rudder, mass 1e-08
- link base_link: geometry collision box size=0.55 2.144 0.05; visual mesh filename=package://standard_vtol/meshes/base_link_visual_0.stl scale=0.001 0.001 0.001
- link left_elevon: geometry visual mesh filename=package://standard_vtol/meshes/left_elevon_visual_0.stl scale=0.001 0.001 0.001
- link right_elevon: geometry visual mesh filename=package://standard_vtol/meshes/right_elevon_visual_0.stl scale=0.001 0.001 0.001
- link rotor_0: geometry collision cylinder length=0.005 radius=0.1; visual mesh filename=package://standard_vtol/meshes/rotor_0_vis.stl scale=1 1 1
- link rotor_1: geometry collision cylinder length=0.005 radius=0.1; visual mesh filename=package://standard_vtol/meshes/rotor_1_vis.stl scale=1 1 1
- link rotor_2: geometry collision cylinder length=0.005 radius=0.1; visual mesh filename=package://standard_vtol/meshes/rotor_2_vis.stl scale=1 1 1
- link rotor_3: geometry collision cylinder length=0.005 radius=0.1; visual mesh filename=package://standard_vtol/meshes/rotor_3_vis.stl scale=1 1 1
- link rotor_4: geometry collision cylinder length=0.005 radius=0.06; visual mesh filename=package://standard_vtol/meshes/rotor_4_vis.stl scale=0.8 0.8 0.8
Joints:
- added joint rudder_joint: type revolute, parent base_link, child rudder, origin xyz=-0.5 0 0.05 rpy=0.00 0 0.0, axis 1 0 0, limit lower=-0.01 upper=0.01 effort=1000 velocity=1000
- joint elevator_joint: limit lower=-0.78 upper=0.78 effort=1000 velocity=1000 -> lower=-0.53 upper=0.53 effort=1000 velocity=1000
- joint left_elevon_joint: limit lower=-0.78 upper=0.78 effort=1000 velocity=1000 -> lower=-0.53 upper=0.53 effort=1000 velocity=1000; origin xyz=-0.18 0.6 -0.005 rpy=0 -0 0.265 -> xyz=-0.18 0.6 -0.005 rpy=0 0 0.265
- joint right_elevon_joint: limit lower=-0.78 upper=0.78 effort=1000 velocity=1000 -> lower=-0.53 upper=0.53 effort=1000 velocity=1000
- joint rotor_4_joint: origin xyz=-0.22 0 0 rpy=0 0 0 -> xyz=-0.22 0 0 rpy=0 1.57 0

File: acesim/env/mujoco/asset/uuv_bluerov2_heavy/uuv_bluerov2_heavy.urdf (robot description, URDF)
Before this commit: robot uuv_bluerov2_heavy, 9 links, 8 joints
Links:
- link base_link: mass 13 -> 11; geometry collision box size=0.45510339736938477 0.5744732022285461 0.25284991040825844; visual mesh filename=package://uuv_bluerov2_heavy/meshes/base_link_visual_0.stl
- link rotor_0: mass 0.05 -> 1e-10
- link rotor_1: mass 0.05 -> 1e-10
- link rotor_2: mass 0.05 -> 1e-10
- link rotor_3: mass 0.05 -> 1e-10
- link rotor_4: mass 0.05 -> 1e-10
- link rotor_5: mass 0.05 -> 1e-10
- link rotor_6: mass 0.05 -> 1e-10
- link rotor_7: mass 0.05 -> 1e-10
Joints:
- joint rotor_0_joint: origin xyz=0.14 -0.1 -0.06 rpy=1.69865416e-10 1.570796 0.785398 -> xyz=0.14 -0.1 0 rpy=0 1.570796 0.78539815
- joint rotor_1_joint: origin xyz=0.14 0.1 -0.06 rpy=-1.69865416e-10 1.570796 -0.785398 -> xyz=0.14 0.1 0 rpy=0 1.570796 -0.78539815
- joint rotor_2_joint: origin xyz=-0.14 -0.1 -0.06 rpy=-1.69865416e-10 1.570796 -0.785398 -> xyz=-0.14 -0.1 0 rpy=0 1.570796 2.356194
- joint rotor_3_joint: origin xyz=-0.14 0.1 -0.06 rpy=1.69865416e-10 1.570796 0.785398 -> xyz=-0.14 0.1 0 rpy=0 1.570796 -2.356194
- joint rotor_4_joint: origin xyz=0.12 -0.22 0 rpy=0 -0 0 -> xyz=0.12 -0.22 0.08 rpy=0 0 0
- joint rotor_5_joint: origin xyz=0.12 0.22 0 rpy=3.1415 -0 0 -> xyz=0.12 0.22 0.08 rpy=0 0 0
- joint rotor_6_joint: origin xyz=-0.12 -0.22 0 rpy=3.1415 -0 0 -> xyz=-0.12 -0.22 0.08 rpy=0 0 0
- joint rotor_7_joint: origin xyz=-0.12 0.22 0 rpy=0 -0 0 -> xyz=-0.12 0.22 0.08 rpy=0 0 0
