Commit message: feat(asset): refresh x500 arm2x MuJoCo asset

File: acesim/env/mujoco/asset/x500_arm2x/x500_arm2x.urdf (robot description, URDF)
Before this commit: robot x500_arm2x, 13 links, 12 joints
Links:
- removed link link_0
- link base_link: mass 0.57465 -> 1.9041
- link gripper_left: mass 0.02118 -> 0.02254
- link gripper_right: mass 0.02118 -> 0.01854
- link link_1: mass 0.09846 -> 0.15156
- link link_2: mass 0.09066 -> 0.14776
- link link_3: mass 0.0449 -> 0.062
- link link_4: mass 0.10644 -> 0.11656
- link link_5: mass 0.0069 -> 0.0035
Joints:
- removed joint joint_0
- removed joint rotor_joint_1
- removed joint rotor_joint_2
- removed joint rotor_joint_3
- removed joint rotor_joint_4
- added joint joint_rotor_1: type continuous, parent base_link, child rotor_1, origin xyz=0.17688 -0.17688 0.0153 rpy=0 0 0, axis 0 0 1, limit effort=0.18 velocity=1032.2
- added joint joint_rotor_2: type continuous, parent base_link, child rotor_2, origin xyz=-0.17688 0.17688 0.0153 rpy=0 0 0, axis 0 0 1, limit effort=0.18 velocity=1032.2
- added joint joint_rotor_3: type continuous, parent base_link, child rotor_3, origin xyz=0.17688 0.17688 0.0153 rpy=0 0 0, axis 0 0 1, limit effort=0.18 velocity=1032.2
- added joint joint_rotor_4: type continuous, parent base_link, child rotor_4, origin xyz=-0.17688 -0.17688 0.0153 rpy=0 0 0, axis 0 0 1, limit effort=0.18 velocity=1032.18
- joint joint_1: limit lower=-2.6485 upper=2.6485 effort=4.9008 velocity=8.95 -> lower=-2.6485 upper=2.6485 effort=5.24 velocity=6.28; origin xyz=0 -0.04611 0 rpy=3.1416 1.5708 0 -> xyz=0 0.0002 -0.1453 rpy=-1.5708 0 3.1416; parent link_0 -> base_link
- joint joint_2: limit lower=0 upper=3.4907 effort=1.3918 velocity=10.47 -> lower=0 upper=3.4907 effort=3.92 velocity=7.85; origin xyz=-0.04068 0.2314 0 rpy=0 0 3.1416 -> xyz=-0.04098 0.2314 -0.0005 rpy=0 0 3.1416
- joint joint_3: limit lower=-2.6485 upper=2.6485 effort=1.3918 velocity=10.47 -> lower=-2.6485 upper=2.6485 effort=2.75 velocity=4.71; origin xyz=-0.04068 -0.24862 0 rpy=0 0 0 -> xyz=-0.04098 -0.26861 0 rpy=0 0 0
- joint joint_4: limit lower=-3.1416 upper=3.1416 effort=1.3918 velocity=10.47 -> lower=-3.1416 upper=3.1416 effort=1.11 velocity=10.47; origin xyz=0 -0.059 0 rpy=1.5708 -1.5708 0 -> xyz=0 -0.05189 0 rpy=1.5708 1.5708 0
- joint joint_5: limit lower=-1.723 upper=0 effort=1.3918 velocity=10.47 -> lower=-1.723 upper=0 effort=1.11 velocity=10.47; origin xyz=0 0 0.0355 rpy=0 0 0 -> xyz=0 0 0.037 rpy=0 0 0
- joint joint_gripper_left: limit lower=-0.04225 upper=0 effort=49.06 velocity=0.0297 -> lower=-0.04225 upper=0 effort=49.06 velocity=0.03; origin xyz=-0.05175 0 0.0602 rpy=-1.5708 0 1.5708 -> xyz=0.04225 0.00825 0.0359 rpy=-1.5708 0 -1.5708; parent link_4 -> link_5
- joint joint_gripper_right: limit lower=0 upper=0.04225 effort=49.06 velocity=0.0297 -> lower=-0.04225 upper=0 effort=49.06 velocity=0.03; mimic joint=joint_gripper_left multiplier=-1 offset=0 -> (none); origin xyz=0.05175 0 0.0602 rpy=-1.5708 0 1.5708 -> xyz=-0.04225 0.00825 0.0359 rpy=-1.5708 0 1.5708; parent link_4 -> link_5

Commit message: feat(sim): update x500 arm2x integration stack
Add ACEFollower-compatible ROS2 command handling, PX4 control and truth streams, raw measurement noise and delay plumbing, refreshed x500_arm2x assets, and calibrated rotor throttle dynamics.

File: acesim/env/mujoco/asset/x500_arm2x/x500_arm2x.urdf (robot description, URDF)
Before this commit: robot x500_arm2x, 12 links, 11 joints
Links:
- link base_link: mass 1.9041 -> 2.20454277
- link gripper_left: mass 0.02254 -> 0.02324
- link gripper_right: mass 0.01854 -> 0.02348
- link link_2: mass 0.14776 -> 0.14766
- link link_3: mass 0.062 -> 0.0636
- link link_4: mass 0.11656 -> 0.1025
- link rotor_1: mass 0.012 -> 0.0132
- link rotor_2: mass 0.012 -> 0.0132
- link rotor_3: mass 0.012 -> 0.0132
- link rotor_4: mass 0.012 -> 0.0132
Joints:
- joint joint_1: origin xyz=0 0.0002 -0.1453 rpy=-1.5708 0 3.1416 -> xyz=0 0.0002 -0.1503 rpy=-1.5708 0 3.1416
- joint joint_2: limit lower=0 upper=3.4907 effort=3.92 velocity=7.85 -> lower=0 upper=3.1415 effort=3.92 velocity=7.85; origin xyz=-0.04098 0.2314 -0.0005 rpy=0 0 3.1416 -> xyz=-0.04123 0.2314 -0.0005 rpy=0 0 3.1416
- joint joint_3: origin xyz=-0.04098 -0.26861 0 rpy=0 0 0 -> xyz=-0.04098 -0.2686 0 rpy=0 0 0
- joint joint_4: limit lower=-3.1416 upper=3.1416 effort=1.11 velocity=10.47 -> lower=-3.1415 upper=3.1415 effort=1.11 velocity=10.47
- joint joint_gripper_left: limit lower=-0.04225 upper=0 effort=49.06 velocity=0.03 -> lower=-0.04225 upper=0 effort=22.7 velocity=0.257; origin xyz=0.04225 0.00825 0.0359 rpy=-1.5708 0 -1.5708 -> xyz=0.040975 0.008255 0.0643 rpy=-1.5708 0 -1.5708; parent link_5 -> link_4
- joint joint_gripper_right: limit lower=-0.04225 upper=0 effort=49.06 velocity=0.03 -> lower=-0.04225 upper=0 effort=22.7 velocity=0.257; origin xyz=-0.04225 0.00825 0.0359 rpy=-1.5708 0 1.5708 -> xyz=-0.040975 0.008255 0.0643 rpy=-1.5708 0 1.5708; parent link_5 -> link_4
- joint joint_rotor_1: origin xyz=0.17688 -0.17688 0.0153 rpy=0 0 0 -> xyz=0.17688 -0.17688 0.0086418 rpy=0 0 0
- joint joint_rotor_2: origin xyz=-0.17688 0.17688 0.0153 rpy=0 0 0 -> xyz=-0.17688 0.17688 0.0086418 rpy=0 0 0
- joint joint_rotor_3: origin xyz=0.17688 0.17688 0.0153 rpy=0 0 0 -> xyz=0.17688 0.17688 0.0086418 rpy=0 0 0
- joint joint_rotor_4: limit effort=0.18 velocity=1032.18 -> effort=0.18 velocity=1032.2; origin xyz=-0.17688 -0.17688 0.0153 rpy=0 0 0 -> xyz=-0.17688 -0.17688 0.0086418 rpy=0 0 0
